File: doc/pcb/flamer/flamer.sch (KiCad schematic (older format))
At the start: 24 parts, among them J1 5V INPUT, J2 SERVO, Q1 BSS138, SW1 REV, U1 LM1117-3.3, U2 STM32L041F6Px

Commit message: 1.1
Parts:
- removed SW1: REV, Connector_PinSocket_2.54mm:PinSocket_1x03_P2.54mm_Vertical, symbol Switch:SW_SPDT
- added C? (x6): 475, symbol Device:C
- added C? (x2): 104, symbol Device:C
- added C?: 475, Capacitor_SMD:C_0603_1608Metric, symbol Device:C
- added L?: 10uH, symbol Device:L
- added R? (x5): 10k, symbol Device:R
- added U?: LM35-D, Package_SO:SOIC-8_3.9x4.9mm_P1.27mm, symbol Sensor_Temperature:LM35-D
- C1: value 105 -> 107
- C2: value 104 -> 107
Connections:
- net +3V3: now also C?.2, L?.1; no longer U2.5 (VDDA)
- net +5V: now also C?.1, C?.1, U?.8 (+VS)
- net GND: now also C?.1, C?.2, C?.2, C?.2, C?.2, C?.2, C?.2, C?.2, C?.2, U?.4 (GND)
- net REG_D: now also C?.1, R?.1; no longer RV4.2
- net REG_I: now also C?.1, R?.1; no longer RV3.2
- net REG_P: now also C?.1, R?.1; no longer RV2.2
- net SET: now also C?.1, R?.1; no longer RV1.2
- net REVERSE renamed TEMPERATURE
- net TEMPERATURE: now also C?.1, C?.1, R?.1
- new net: L?.2, U2.5 (VDDA)
- new net: R?.2, RV1.2
- new net: R?.2, RV2.2
- new net: R?.2, RV3.2
- new net: R?.2, RV4.2
- new net: R?.2, U?.1 (Vout)
Other:
- moved on the sheet: C5, C6, RV1, RV2, RV3
